File: ecad/IOBoard/IOBoard.kicad_pcb (KiCad board)
At the start: 2 copper layers, 34.6 x 88.7 mm, 11 parts, among them J1 SN37A12B, J2 PJ-102A, J3 toEffectsBoard, J4 SN37A12A, U1 FS57003PLT2B2M2QE

Commit message: Update before switch to single-board design
Parts:
- removed BAT1: BC9VPC, DigiKey:PinHeader_1x2_P2.54mm
- D1: value LED -> QBL8XX60D
- J1: value SN37A12B -> ACJM-HHDR; footprint screaming-panda:Switchcraft_SN37A12B -> screaming-panda:ACJM-HHDR
- J4: value SN37A12A -> ACJM-HHDR; footprint screaming-panda:Switchcraft_SN37A12A -> screaming-panda:ACJM-HHDR
- moved J1 29.8 mm to (94.3, 117.6)
- moved C3 19.1 mm to (92.2, 66.2), turned to 0 degrees
- moved J3 18.6 mm to (99.9, 79.3)
- moved C2 17.7 mm to (92.2, 64.2), turned to 0 degrees
- moved C1 16.7 mm to (92.2, 62.2), turned to 0 degrees
- moved R1 15.8 mm to (106.0, 105.8)
- moved D1 15.7 mm to (98.4, 105.8)
- moved J4 15.3 mm to (106.0, 93.8)
- moved J2 3.97 mm to (100.0, 64.4)
- moved U1 0.11 mm to (100.0, 135.7)
Connections:
- J1 pad T: /SIG_IN -> /PassThru
- J2 pad 3: Net-(BAT1-PadPOS) -> GND
- U1 pad 4: /SIG_IN -> /PassThru
- U1 pad 9: /SIG_IN -> /PassThru
Routing:
- net /SIG_IN: track 83.4 -> 0.00 mm
- net /EFFECT_OUT: track 73.1 -> 0.00 mm
- net Net-(BAT1-PadNEG): track 27.1 -> 0.00 mm
- net Net-(D1-Pad1): track 23.1 -> 37.8 mm
- net Net-(BAT1-PadPOS): track 6.42 -> 0.00 mm
- net GND: track 10.4 -> 12.0 mm
- added copper zone on F.Cu, net +9V
- added copper zone on B.Cu, net GND
