File: ecad/IOBoard/IOBoard.sch (KiCad schematic (older format))
At the start: 11 parts, among them J1 SN37A12B, J2 PJ-102A, J3 toEffectsBoard, J4 SN37A12A, U1 FS57003PLT2B2M2QE

Commit message: Rearrange schematics
Other:
- moved on the sheet: R1
Changed lines of the file:
@@
 L Device:R R1
 U 1 1 60060421
-P 1950 2300
-F 0 "R1" H 2020 2346 50  0000 L CNN
-F 1 "1k" H 2020 2255 50  0000 L CNN
-F 2 "Resistor_SMD:R_0805_2012Metric_Pad1.20x1.40mm_HandSolder" V 1880 2300 50  0001 C CNN
-F 3 "~" H 1950 2300 50  0001 C CNN
-F 4 "R" H 1950 2300 50  0001 C CNN "Spice_Primitive"
-F 5 "1k" H 1950 2300 50  0001 C CNN "Spice_Model"
-F 6 "Y" H 1950 2300 50  0001 C CNN "Spice_Netlist_Enabled"
-	1    1950 2300
+P 2000 2300
+F 0 "R1" H 2070 2346 50  0000 L CNN
+F 1 "1k" H 2070 2255 50  0000 L CNN
+F 2 "Resistor_SMD:R_0805_2012Metric_Pad1.20x1.40mm_HandSolder" V 1930 2300 50  0001 C CNN
+F 3 "~" H 2000 2300 50  0001 C CNN
+F 4 "R" H 2000 2300 50  0001 C CNN "Spice_Primitive"
+F 5 "1k" H 2000 2300 50  0001 C CNN "Spice_Model"
+F 6 "Y" H 2000 2300 50  0001 C CNN "Spice_Netlist_Enabled"
+	1    2000 2300
 	1    0    0    -1
 $EndComp
 Wire Wire Line
-	1950 2500 1900 2500
+	2000 2500 1900 2500
 Wire Wire Line
-	1950 2450 1950 2500
+	2000 2450 2000 2500
 Wire Wire Line
 	1100 1750 1250 1750
@@
 	1350 2600 1400 2600
 Wire Wire Line
-	1950 2100 1950 2150
+	2000 2100 2000 2150
 $Comp
 L power:+9V #PWR0110
 U 1 1 600618E7
-P 1950 2100
-F 0 "#PWR0110" H 1950 1950 50  0001 C CNN
-F 1 "+9V" H 1965 2273 50  0000 C CNN
-F 2 "" H 1950 2100 50  0001 C CNN
-F 3 "" H 1950 2100 50  0001 C CNN
-	1    1950 2100
+P 2000 2100
+F 0 "#PWR0110" H 2000 1950 50  0001 C CNN
+F 1 "+9V" H 2015 2273 50  0000 C CNN
+F 2 "" H 2000 2100 50  0001 C CNN
+F 3 "" H 2000 2100 50  0001 C CNN
+	1    2000 2100
 	1    0    0    -1
 $EndComp

Commit message: Update before switch to single-board design
Parts:
- removed BAT1: BC9VPC, DigiKey:PinHeader_1x2_P2.54mm, symbol dk_Battery-Holders-Clips-Contacts:BC9VPC
- removed J1: SN37A12B, screaming-panda:Switchcraft_SN37A12B, symbol screaming-panda:SN37A12B
- removed J4: SN37A12A, screaming-panda:Switchcraft_SN37A12A, symbol screaming-panda:SN37A12A
- added J1, J4: ACJM-HHDR, screaming-panda:ACJM-HHDR, symbol Connector:AudioJack2_Switch
Connections:
- net GND: now also J2.3, J1.S, J1.SN, J1.TN, J4.S
- net SIG_IN: no longer U1.4, U1.9
- net SIG_OUT: now also J4.T
- new net PassThru: J1.T, U1.4, U1.9
- no-connect marks 0 -> 2
Other:
- moved on the sheet: C1, C2, C3, D1, J2, J3, R1, U1A, U1B, U1C
