File: ecad/EffectsBoard/EffectsBoard.sch (KiCad schematic (older format))
At the start: 8 parts, among them J1 toIOBoard, U1 RC4558

Commit message: Rearrange schematics
Other:
- moved on the sheet: U1C
Changed lines of the file:
@@
 L Amplifier_Operational:RC4558 U1
 U 3 1 60246CA0
-P 3450 1150
-F 0 "U1" H 3408 1196 50  0000 L CNN
-F 1 "RC4558" H 3408 1105 50  0000 L CNN
-F 2 "" H 3450 1150 50  0001 C CNN
-F 3 "http://www.ti.com/lit/ds/symlink/rc4558.pdf" H 3450 1150 50  0001 C CNN
-	3    3450 1150
+P 3450 1100
+F 0 "U1" H 3408 1146 50  0000 L CNN
+F 1 "RC4558" H 3408 1055 50  0000 L CNN
+F 2 "" H 3450 1100 50  0001 C CNN
+F 3 "http://www.ti.com/lit/ds/symlink/rc4558.pdf" H 3450 1100 50  0001 C CNN
+	3    3450 1100
 	1    0    0    -1
 $EndComp
@@
 L power:+9V #PWR0110
 U 1 1 6025900B
-P 3350 750
-F 0 "#PWR0110" H 3350 600 50  0001 C CNN
-F 1 "+9V" H 3365 923 50  0000 C CNN
-F 2 "" H 3350 750 50  0001 C CNN
-F 3 "" H 3350 750 50  0001 C CNN
-	1    3350 750
+P 3350 700
+F 0 "#PWR0110" H 3350 550 50  0001 C CNN
+F 1 "+9V" H 3365 873 50  0000 C CNN
+F 2 "" H 3350 700 50  0001 C CNN
+F 3 "" H 3350 700 50  0001 C CNN
+	1    3350 700
 	1    0    0    -1
 $EndComp
 Wire Wire Line
-	3350 750  3350 850
+	3350 700  3350 800
 Wire Wire Line
-	3350 1450 3350 1550
+	3350 1400 3350 1550
 $Sheet
 S 1500 3500 500  500

Commit message: Update ecad autosave
Parts:
- C1, C2, C3: footprint (none) -> Capacitor_SMD:C_0805_2012Metric_Pad1.18x1.45mm_HandSolder
- J1: footprint (none) -> Connector_PinSocket_1.27mm:PinSocket_2x02_P1.27mm_Vertical
- R1, R2: footprint (none) -> Resistor_SMD:R_0805_2012Metric_Pad1.20x1.40mm_HandSolder
- U1: footprint (none) -> Package_SO:Texas_R-PDSO-G8_EP2.95x4.9mm_Mask2.4x3.1mm
Changed lines of the file:
@@
 F 0 "J1" H 1100 967 50  0000 C CNN
 F 1 "toIOBoard" H 1100 876 50  0000 C CNN
-F 2 "" H 1050 750 50  0001 C CNN
+F 2 "Connector_PinSocket_1.27mm:PinSocket_2x02_P1.27mm_Vertical" H 1050 750 50  0001 C CNN
 F 3 "~" H 1050 750 50  0001 C CNN
 	1    1050 750
@@
 F 0 "C1" H 2200 1050 50  0000 L CNN
 F 1 "100u" H 2200 850 50  0000 L CNN
-F 2 "" H 2238 800 50  0001 C CNN
+F 2 "Capacitor_SMD:C_0805_2012Metric_Pad1.18x1.45mm_HandSolder" H 2238 800 50  0001 C CNN
 F 3 "~" H 2200 950 50  0001 C CNN
 	1    2200 950
@@
 F 0 "C2" H 2400 1050 50  0000 L CNN
 F 1 "10n" H 2400 850 50  0000 L CNN
-F 2 "" H 2438 800 50  0001 C CNN
+F 2 "Capacitor_SMD:C_0805_2012Metric_Pad1.18x1.45mm_HandSolder" H 2438 800 50  0001 C CNN
 F 3 "~" H 2400 950 50  0001 C CNN
 	1    2400 950
@@
 F 0 "R1" H 2720 996 50  0000 L CNN
 F 1 "10k" H 2720 905 50  0000 L CNN
-F 2 "" V 2580 950 50  0001 C CNN
+F 2 "Resistor_SMD:R_0805_2012Metric_Pad1.20x1.40mm_HandSolder" V 2580 950 50  0001 C CNN
 F 3 "~" H 2650 950 50  0001 C CNN
 	1    2650 950
@@
 F 0 "R2" H 2720 1396 50  0000 L CNN
 F 1 "10k" H 2720 1305 50  0000 L CNN
-F 2 "" V 2580 1350 50  0001 C CNN
+F 2 "Resistor_SMD:R_0805_2012Metric_Pad1.20x1.40mm_HandSolder" V 2580 1350 50  0001 C CNN
 F 3 "~" H 2650 1350 50  0001 C CNN
 	1    2650 1350
@@
 F 0 "C3" H 3068 1396 50  0000 L CNN
 F 1 "47u" H 3068 1305 50  0000 L CNN
-F 2 "" H 2988 1200 50  0001 C CNN
+F 2 "Capacitor_SMD:C_0805_2012Metric_Pad1.18x1.45mm_HandSolder" H 2988 1200 50  0001 C CNN
 F 3 "~" H 2950 1350 50  0001 C CNN
 	1    2950 1350
@@
 F 0 "U1" H 3408 1146 50  0000 L CNN
 F 1 "RC4558" H 3408 1055 50  0000 L CNN
-F 2 "" H 3450 1100 50  0001 C CNN
+F 2 "Package_SO:Texas_R-PDSO-G8_EP2.95x4.9mm_Mask2.4x3.1mm" H 3450 1100 50  0001 C CNN
 F 3 "http://www.ti.com/lit/ds/symlink/rc4558.pdf" H 3450 1100 50  0001 C CNN
 	3    3450 1100
