File: ecad/EffectsBoard/volume.sch (KiCad schematic (older format))
At the start: 10 parts, among them Q2 2N4401BU

Commit message: Rearrange schematics
Other:
- moved on the sheet: C10, C8, C9, Q2, R13, R14, R15, R16, R17, RV3

Commit message: Update ecad autosave
Parts:
- C10, C8, C9: footprint (none) -> Capacitor_SMD:C_0805_2012Metric_Pad1.18x1.45mm_HandSolder
- R13, R14, R15, R16, R17: footprint (none) -> Resistor_SMD:R_0805_2012Metric_Pad1.20x1.40mm_HandSolder
- RV3: footprint (none) -> screaming-panda:Potentiometer_Bourns_PTV09A-1_Single_Vertical
Changed lines of the file:
@@
 F 0 "C8" V 898 950 50  0000 C CNN
 F 1 "1u" V 989 950 50  0000 C CNN
-F 2 "" H 1188 800 50  0001 C CNN
+F 2 "Capacitor_SMD:C_0805_2012Metric_Pad1.18x1.45mm_HandSolder" H 1188 800 50  0001 C CNN
 F 3 "~" H 1150 950 50  0001 C CNN
 	1    1150 950
@@
 F 0 "R13" V 1293 950 50  0000 C CNN
 F 1 "1k" V 1384 950 50  0000 C CNN
-F 2 "" V 1430 950 50  0001 C CNN
+F 2 "Resistor_SMD:R_0805_2012Metric_Pad1.20x1.40mm_HandSolder" V 1430 950 50  0001 C CNN
 F 3 "~" H 1500 950 50  0001 C CNN
 	1    1500 950
@@
 F 0 "RV3" V 1750 1050 50  0000 R CNN
 F 1 "100ka" V 1650 1050 50  0000 R CNN
-F 2 "" H 1850 950 50  0001 C CNN
+F 2 "screaming-panda:Potentiometer_Bourns_PTV09A-1_Single_Vertical" H 1850 950 50  0001 C CNN
 F 3 "~" H 1850 950 50  0001 C CNN
 	1    1850 950
@@
 F 0 "C9" V 1948 950 50  0000 C CNN
 F 1 "0u1" V 2039 950 50  0000 C CNN
-F 2 "" H 2238 800 50  0001 C CNN
+F 2 "Capacitor_SMD:C_0805_2012Metric_Pad1.18x1.45mm_HandSolder" H 2238 800 50  0001 C CNN
 F 3 "~" H 2200 950 50  0001 C CNN
 	1    2200 950
@@
 F 0 "R14" H 2470 1446 50  0000 L CNN
 F 1 "501k" H 2470 1355 50  0000 L CNN
-F 2 "" V 2330 1400 50  0001 C CNN
+F 2 "Resistor_SMD:R_0805_2012Metric_Pad1.20x1.40mm_HandSolder" V 2330 1400 50  0001 C CNN
 F 3 "~" H 2400 1400 50  0001 C CNN
 	1    2400 1400
@@
 F 0 "R15" H 2820 1446 50  0000 L CNN
 F 1 "10k" H 2820 1355 50  0000 L CNN
-F 2 "" V 2680 1400 50  0001 C CNN
+F 2 "Resistor_SMD:R_0805_2012Metric_Pad1.20x1.40mm_HandSolder" V 2680 1400 50  0001 C CNN
 F 3 "~" H 2750 1400 50  0001 C CNN
 	1    2750 1400
@@
 F 0 "R16" V 3243 1200 50  0000 C CNN
 F 1 "100" V 3334 1200 50  0000 C CNN
-F 2 "" V 3380 1200 50  0001 C CNN
+F 2 "Resistor_SMD:R_0805_2012Metric_Pad1.20x1.40mm_HandSolder" V 3380 1200 50  0001 C CNN
 F 3 "~" H 3450 1200 50  0001 C CNN
 	1    3450 1200
@@
 F 0 "C10" V 4055 1200 50  0000 C CNN
 F 1 "CP" V 3964 1200 50  0000 C CNN
-F 2 "" H 3838 1050 50  0001 C CNN
+F 2 "Capacitor_SMD:C_0805_2012Metric_Pad1.18x1.45mm_HandSolder" H 3838 1050 50  0001 C CNN
 F 3 "~" H 3800 1200 50  0001 C CNN
 	1    3800 1200
@@
 F 0 "R17" H 4070 1446 50  0000 L CNN
 F 1 "10k" H 4070 1355 50  0000 L CNN
-F 2 "" V 3930 1400 50  0001 C CNN
+F 2 "Resistor_SMD:R_0805_2012Metric_Pad1.20x1.40mm_HandSolder" V 3930 1400 50  0001 C CNN
 F 3 "~" H 4000 1400 50  0001 C CNN
 	1    4000 1400
