File: ecad/PotBoard/PotBoard.sch (KiCad schematic (older format))
At the start: 6 parts, among them J1 DrivePot, J2 TonePot, J3 VolumePot

Commit message: Clean up ecad
Parts:
- J1, J2, J3: manf# (none) -> C031LFBN-RC
- RV1: manf# (none) -> PTV09A-4020F-A504
- RV2: manf# (none) -> PTV09A-4020F-B203
- RV3: value 100ka -> 20ka; manf# (none) -> PTV09A-4020F-A203
Changed lines of the file:
@@
 F 1 "500ka" V 634 750 50  0000 C CNN
 F 2 "screaming-panda:Potentiometer_Bourns_PTV09A-1_Single_Vertical" H 750 750 50  0001 C CNN
-F 3 "~" H 750 750 50  0001 C CNN
+F 3 "https://www.bourns.com/docs/Product-Datasheets/PTV09.pdf" H 750 750 50  0001 C CNN
+F 4 "PTV09A-4020F-A504" H 750 750 50  0001 C CNN "manf#"
 	1    750  750
 	0    -1   1    0
@@
 F 1 "20kb" V 1134 750 50  0000 C CNN
 F 2 "screaming-panda:Potentiometer_Bourns_PTV09A-1_Single_Vertical" H 1250 750 50  0001 C CNN
-F 3 "~" H 1250 750 50  0001 C CNN
+F 3 "https://www.bourns.com/docs/Product-Datasheets/PTV09.pdf" H 1250 750 50  0001 C CNN
+F 4 "PTV09A-4020F-B203" H 1250 750 50  0001 C CNN "manf#"
 	1    1250 750
 	0    -1   1    0
@@
 P 1750 750
 F 0 "RV3" V 1543 750 50  0000 C CNN
-F 1 "100ka" V 1634 750 50  0000 C CNN
+F 1 "20ka" V 1634 750 50  0000 C CNN
 F 2 "screaming-panda:Potentiometer_Bourns_PTV09A-1_Single_Vertical" H 1750 750 50  0001 C CNN
-F 3 "~" H 1750 750 50  0001 C CNN
+F 3 "https://www.bourns.com/docs/Product-Datasheets/PTV09.pdf" H 1750 750 50  0001 C CNN
+F 4 "PTV09A-4020F-A203" H 1750 750 50  0001 C CNN "manf#"
 	1    1750 750
 	0    -1   1    0
@@
 F 1 "DrivePot" V 800 1450 50  0000 R CNN
 F 2 "Connector_PinSocket_2.00mm:PinSocket_1x03_P2.00mm_Vertical" H 750 1300 50  0001 C CNN
-F 3 "~" H 750 1300 50  0001 C CNN
+F 3 "https://media.digikey.com/pdf/Data%20Sheets/Sullins%20PDFs/Female_Headers.100_DS.pdf" H 750 1300 50  0001 C CNN
+F 4 "C031LFBN-RC" H 750 1300 50  0001 C CNN "manf#"
 	1    750  1300
 	0    -1   1    0
@@
 F 1 "TonePot" V 1300 1450 50  0000 R CNN
 F 2 "Connector_PinSocket_2.00mm:PinSocket_1x03_P2.00mm_Vertical" H 1250 1300 50  0001 C CNN
-F 3 "~" H 1250 1300 50  0001 C CNN
+F 3 "https://media.digikey.com/pdf/Data%20Sheets/Sullins%20PDFs/Female_Headers.100_DS.pdf" H 1250 1300 50  0001 C CNN
+F 4 "C031LFBN-RC" H 1250 1300 50  0001 C CNN "manf#"
 	1    1250 1300
 	0    -1   1    0
@@
 F 1 "VolumePot" V 1800 1500 50  0000 R CNN
 F 2 "Connector_PinSocket_2.00mm:PinSocket_1x03_P2.00mm_Vertical" H 1750 1300 50  0001 C CNN
-F 3 "~" H 1750 1300 50  0001 C CNN
+F 3 "https://media.digikey.com/pdf/Data%20Sheets/Sullins%20PDFs/Female_Headers.100_DS.pdf" H 1750 1300 50  0001 C CNN
+F 4 "C031LFBN-RC" H 1750 1300 50  0001 C CNN "manf#"
 	1    1750 1300
 	0    -1   1    0

Commit message: Update ecad BOM
Change transistor to 2N4424
Parts:
- J1, J2, J3: MPN (none) -> C031LFBN-RC
- RV1: MPN (none) -> PTV09A-4020F-A504
- RV2: MPN (none) -> PTV09A-4020F-B203
- RV3: MPN (none) -> PTV09A-4020F-A203
Changed lines of the file:
@@
 F 3 "https://www.bourns.com/docs/Product-Datasheets/PTV09.pdf" H 750 750 50  0001 C CNN
 F 4 "PTV09A-4020F-A504" H 750 750 50  0001 C CNN "manf#"
+F 5 "PTV09A-4020F-A504" H 750 750 50  0001 C CNN "MPN"
 	1    750  750
 	0    -1   1    0
@@
 F 3 "https://www.bourns.com/docs/Product-Datasheets/PTV09.pdf" H 1250 750 50  0001 C CNN
 F 4 "PTV09A-4020F-B203" H 1250 750 50  0001 C CNN "manf#"
+F 5 "PTV09A-4020F-B203" H 1250 750 50  0001 C CNN "MPN"
 	1    1250 750
 	0    -1   1    0
@@
 F 3 "https://www.bourns.com/docs/Product-Datasheets/PTV09.pdf" H 1750 750 50  0001 C CNN
 F 4 "PTV09A-4020F-A203" H 1750 750 50  0001 C CNN "manf#"
+F 5 "PTV09A-4020F-A203" H 1750 750 50  0001 C CNN "MPN"
 	1    1750 750
 	0    -1   1    0
@@
 F 3 "https://media.digikey.com/pdf/Data%20Sheets/Sullins%20PDFs/Female_Headers.100_DS.pdf" H 750 1300 50  0001 C CNN
 F 4 "C031LFBN-RC" H 750 1300 50  0001 C CNN "manf#"
+F 5 "C031LFBN-RC" H 750 1300 50  0001 C CNN "MPN"
 	1    750  1300
 	0    -1   1    0
@@
 F 3 "https://media.digikey.com/pdf/Data%20Sheets/Sullins%20PDFs/Female_Headers.100_DS.pdf" H 1250 1300 50  0001 C CNN
 F 4 "C031LFBN-RC" H 1250 1300 50  0001 C CNN "manf#"
+F 5 "C031LFBN-RC" H 1250 1300 50  0001 C CNN "MPN"
 	1    1250 1300
 	0    -1   1    0
@@
 F 3 "https://media.digikey.com/pdf/Data%20Sheets/Sullins%20PDFs/Female_Headers.100_DS.pdf" H 1750 1300 50  0001 C CNN
 F 4 "C031LFBN-RC" H 1750 1300 50  0001 C CNN "manf#"
+F 5 "C031LFBN-RC" H 1750 1300 50  0001 C CNN "MPN"
 	1    1750 1300
 	0    -1   1    0

Commit message: Update layouts with finished mcad
Parts:
- J1, J2, J3: footprint Connector_PinSocket_2.00mm:PinSocket_1x03_P2.00mm_Vertical -> screaming-panda:C031LFBN-RC
Changed lines of the file:
@@
 encoding utf-8
 Sheet 1 1
-Title ""
-Date ""
-Rev ""
-Comp ""
+Title "Screaming Panda - Pot Board"
+Date "2021-08-24"
+Rev "1.0"
+Comp "John McAvoy"
 Comment1 ""
 Comment2 ""
@@
 F 0 "J1" V 700 1550 50  0000 R CNN
 F 1 "DrivePot" V 800 1450 50  0000 R CNN
-F 2 "Connector_PinSocket_2.00mm:PinSocket_1x03_P2.00mm_Vertical" H 750 1300 50  0001 C CNN
+F 2 "screaming-panda:C031LFBN-RC" H 750 1300 50  0001 C CNN
 F 3 "https://media.digikey.com/pdf/Data%20Sheets/Sullins%20PDFs/Female_Headers.100_DS.pdf" H 750 1300 50  0001 C CNN
 F 4 "C031LFBN-RC" H 750 1300 50  0001 C CNN "manf#"
@@
 F 0 "J2" V 1200 1500 50  0000 R CNN
 F 1 "TonePot" V 1300 1450 50  0000 R CNN
-F 2 "Connector_PinSocket_2.00mm:PinSocket_1x03_P2.00mm_Vertical" H 1250 1300 50  0001 C CNN
+F 2 "screaming-panda:C031LFBN-RC" H 1250 1300 50  0001 C CNN
 F 3 "https://media.digikey.com/pdf/Data%20Sheets/Sullins%20PDFs/Female_Headers.100_DS.pdf" H 1250 1300 50  0001 C CNN
 F 4 "C031LFBN-RC" H 1250 1300 50  0001 C CNN "manf#"
@@
 F 0 "J3" V 1700 1500 50  0000 R CNN
 F 1 "VolumePot" V 1800 1500 50  0000 R CNN
-F 2 "Connector_PinSocket_2.00mm:PinSocket_1x03_P2.00mm_Vertical" H 1750 1300 50  0001 C CNN
+F 2 "screaming-panda:C031LFBN-RC" H 1750 1300 50  0001 C CNN
 F 3 "https://media.digikey.com/pdf/Data%20Sheets/Sullins%20PDFs/Female_Headers.100_DS.pdf" H 1750 1300 50  0001 C CNN
 F 4 "C031LFBN-RC" H 1750 1300 50  0001 C CNN "manf#"
