File: ecad/MainBoard/drive.sch (KiCad schematic (older format))
At the start: 13 parts, among them IC1 RC4558

Commit message: Change to using kicad-library submodule
Parts:
- D1, D2: Spice_Lib_File ../lib/spice_models/1N914.lib -> ../lib/kicad-library/spice_models/1N914.lib
- IC1: Spice_Lib_File ../lib/spice_models/RC4558.301.lib -> ../lib/kicad-library/spice_models/RC4558.301.lib
- R19: Spice_Lib_File ../lib/spice_models/pots.lib -> ../lib/kicad-library/spice_models/pots.lib
Changed lines of the file:
@@
 F 5 "RC4558" H 1700 1800 50  0001 C CNN "Spice_Model"
 F 6 "Y" H 1700 1800 50  0001 C CNN "Spice_Netlist_Enabled"
-F 7 "../lib/spice_models/RC4558.301.lib" H 1700 1800 50  0001 C CNN "Spice_Lib_File"
+F 7 "../lib/kicad-library/spice_models/RC4558.301.lib" H 1700 1800 50  0001 C CNN "Spice_Lib_File"
 F 8 "296-9650-5-ND" H 1700 1800 50  0001 C CNN "Digi-Key_PN"
 F 9 "RC4558D" H 1700 1800 50  0001 C CNN "MPN"
@@
 F 5 "D1N914" H 1700 1100 50  0001 C CNN "Spice_Model"
 F 6 "Y" H 1700 1100 50  0001 C CNN "Spice_Netlist_Enabled"
-F 7 "../lib/spice_models/1N914.lib" H 1700 1100 50  0001 C CNN "Spice_Lib_File"
+F 7 "../lib/kicad-library/spice_models/1N914.lib" H 1700 1100 50  0001 C CNN "Spice_Lib_File"
 F 8 "2 1" H 1700 1100 50  0001 C CNN "Spice_Node_Sequence"
 F 9 "1N914MS-ND" H 1700 1100 50  0001 C CNN "Digi-Key_PN"
@@
 F 2 "Diode_THT:D_DO-35_SOD27_P5.08mm_Vertical_KathodeUp" H 1700 1075 50  0001 C CNN
 F 3 "https://datasheet.octopart.com/1N914-ON-Semiconductor-datasheet-42765246.pdf" H 1700 1250 50  0001 C CNN
-F 4 "../lib/spice_models/1N914.lib" H 1700 1250 50  0001 C CNN "Spice_Lib_File"
+F 4 "../lib/kicad-library/spice_models/1N914.lib" H 1700 1250 50  0001 C CNN "Spice_Lib_File"
 F 5 "D" H 1700 1250 50  0001 C CNN "Spice_Primitive"
 F 6 "D1N914" H 1700 1250 50  0001 C CNN "Spice_Model"
@@
 F 5 "POTDrive" H 1750 700 50  0001 C CNN "Spice_Model"
 F 6 "Y" H 1750 700 50  0001 C CNN "Spice_Netlist_Enabled"
-F 7 "../lib/spice_models/pots.lib" H 1750 700 50  0001 C CNN "Spice_Lib_File"
+F 7 "../lib/kicad-library/spice_models/pots.lib" H 1750 700 50  0001 C CNN "Spice_Lib_File"
 F 8 "Drive Pot" V 1575 725 50  0000 C CNN "Category"
 F 9 "75160-195-08LF" H 1750 700 50  0001 C CNN "Digi-Key_PN"
