File: ecad/MainBoard/gain.sch (KiCad schematic (older format))
At the start: 6 parts, among them Q1 2N4401BU

Commit message: Update BOM and SPIRCE SIM
Add netlist to calculate power dissipation through each resistor
Parts:
- C1: Digi-Key_PN (none) -> 399-C0402C224M8RACTUTR-ND; MPN (none) -> 399-C0402C224M8RACTUTR-ND
- Q1: MPN 2N4401BU -> 2N4401-ND
- R1: Digi-Key_PN (none) -> A130048TR-ND; MPN (none) -> CRGCQ0402J1K0
- R2: Digi-Key_PN (none) -> 2019-RN73R2ATTD5053F100TR-ND; MPN (none) -> RN73R2ATTD5053F100
- R22: Digi-Key_PN (none) -> 10-ERJ-U02J155XTR-ND; MPN (none) -> ERJ-U02J155X
- R3: Digi-Key_PN (none) -> RG2012N-474-W-T1; MPN (none) -> RG20N470KWTR-ND
Changed lines of the file:
@@
 F 1 "1M5" H 820 1255 50  0000 L CNN
 F 2 "Resistor_SMD:R_0805_2012Metric_Pad1.20x1.40mm_HandSolder" V 680 1300 50  0001 C CNN
-F 3 "~" H 750 1300 50  0001 C CNN
+F 3 "https://industrial.panasonic.com/cdbs/www-data/pdf/RDP0000/AOA0000C334.pdf" H 750 1300 50  0001 C CNN
 F 4 "R" H 750 1300 50  0001 C CNN "Spice_Primitive"
 F 5 "1.5Meg" H 750 1300 50  0001 C CNN "Spice_Model"
 F 6 "Y" H 750 1300 50  0001 C CNN "Spice_Netlist_Enabled"
+F 7 "10-ERJ-U02J155XTR-ND" H 750 1300 50  0001 C CNN "Digi-Key_PN"
+F 8 "ERJ-U02J155X" H 750 1300 50  0001 C CNN "MPN"
 	1    750  1300
 	1    0    0    -1
@@
 F 2 "Capacitor_SMD:C_0805_2012Metric_Pad1.18x1.45mm_HandSolder" H 1038 950 50  0001 C CNN
 F 3 "~" H 1000 1100 50  0001 C CNN
+F 4 "399-C0402C224M8RACTUTR-ND" H 1000 1100 50  0001 C CNN "Digi-Key_PN"
+F 5 "399-C0402C224M8RACTUTR-ND" H 1000 1100 50  0001 C CNN "MPN"
 	1    1000 1100
 	0    1    1    0
@@
 F 2 "Resistor_SMD:R_0805_2012Metric_Pad1.20x1.40mm_HandSolder" V 1280 1100 50  0001 C CNN
 F 3 "~" H 1350 1100 50  0001 C CNN
+F 4 "A130048TR-ND" H 1350 1100 50  0001 C CNN "Digi-Key_PN"
+F 5 "CRGCQ0402J1K0" H 1350 1100 50  0001 C CNN "MPN"
 	1    1350 1100
 	0    1    1    0
@@
 F 2 "Resistor_SMD:R_0805_2012Metric_Pad1.20x1.40mm_HandSolder" V 1480 900 50  0001 C CNN
 F 3 "~" H 1550 900 50  0001 C CNN
+F 4 "2019-RN73R2ATTD5053F100TR-ND" H 1550 900 50  0001 C CNN "Digi-Key_PN"
+F 5 "RN73R2ATTD5053F100" H 1550 900 50  0001 C CNN "MPN"
 	1    1550 900
 	1    0    0    -1
@@
 F 3 "https://www.onsemi.com/pub/Collateral/MMBT4401-D.PDF" H 2050 1400 60  0001 L CNN
 F 4 "2N4401-ND" H 2050 1500 60  0001 L CNN "Digi-Key_PN"
-F 5 "2N4401BU" H 2050 1600 60  0001 L CNN "MPN"
+F 5 "2N4401-ND" H 2050 1600 60  0001 L CNN "MPN"
 F 6 "Discrete Semiconductor Products" H 2050 1700 60  0001 L CNN "Category"
 F 7 "Transistors - Bipolar (BJT) - Single" H 2050 1800 60  0001 L CNN "Family"
@@
 F 2 "Resistor_SMD:R_0805_2012Metric_Pad1.20x1.40mm_HandSolder" V 1880 1550 50  0001 C CNN
 F 3 "~" H 1950 1550 50  0001 C CNN
+F 4 "RG2012N-474-W-T1" H 1950 1550 50  0001 C CNN "Digi-Key_PN"
+F 5 "RG20N470KWTR-ND" H 1950 1550 50  0001 C CNN "MPN"
 	1    1950 1550
 	1    0    0    -1

Commit message: Clean up ecad
Parts:
- C1: footprint Capacitor_SMD:C_0805_2012Metric_Pad1.18x1.45mm_HandSolder -> Capacitor_SMD:C_0402_1005Metric_Pad0.74x0.62mm_HandSolder
- R1, R22: footprint Resistor_SMD:R_0805_2012Metric_Pad1.20x1.40mm_HandSolder -> Resistor_SMD:R_0402_1005Metric_Pad0.72x0.64mm_HandSolder
- R2: value 501k -> 505k
Changed lines of the file:
@@
 encoding utf-8
 Sheet 5 5
-Title "Effects Board"
-Date "2021-01-17"
-Rev "1.0"
-Comp "Panda Pals"
-Comment1 "John McAvoy"
+Title "Screaming Panda Guitar Pedal"
+Date "2021-08-08"
+Rev "1v0"
+Comp "John McAvoy"
+Comment1 ""
 Comment2 ""
 Comment3 ""
@@
 AR Path="/60306390/6030F08B" Ref="R22"  Part="1"
 F 0 "R22" H 820 1346 50  0000 L CNN
-F 1 "1M5" H 820 1255 50  0000 L CNN
-F 2 "Resistor_SMD:R_0805_2012Metric_Pad1.20x1.40mm_HandSolder" V 680 1300 50  0001 C CNN
+F 1 "1M5" V 750 1225 50  0000 L CNN
+F 2 "Resistor_SMD:R_0402_1005Metric_Pad0.72x0.64mm_HandSolder" V 680 1300 50  0001 C CNN
 F 3 "https://industrial.panasonic.com/cdbs/www-data/pdf/RDP0000/AOA0000C334.pdf" H 750 1300 50  0001 C CNN
 F 4 "R" H 750 1300 50  0001 C CNN "Spice_Primitive"
@@
 F 0 "C1" V 748 1100 50  0000 C CNN
 F 1 "20n" V 839 1100 50  0000 C CNN
-F 2 "Capacitor_SMD:C_0805_2012Metric_Pad1.18x1.45mm_HandSolder" H 1038 950 50  0001 C CNN
-F 3 "~" H 1000 1100 50  0001 C CNN
+F 2 "Capacitor_SMD:C_0402_1005Metric_Pad0.74x0.62mm_HandSolder" H 1038 950 50  0001 C CNN
+F 3 "https://api.kemet.com/component-edge/download/datasheet/C0402C224M8RACTU.pdf" H 1000 1100 50  0001 C CNN
 F 4 "399-C0402C224M8RACTUTR-ND" H 1000 1100 50  0001 C CNN "Digi-Key_PN"
 F 5 "399-C0402C224M8RACTUTR-ND" H 1000 1100 50  0001 C CNN "MPN"
@@
 AR Path="/6030F0A3" Ref="R?"  Part="1"
 AR Path="/60306390/6030F0A3" Ref="R1"  Part="1"
-F 0 "R1" V 1143 1100 50  0000 C CNN
-F 1 "1k" V 1234 1100 50  0000 C CNN
-F 2 "Resistor_SMD:R_0805_2012Metric_Pad1.20x1.40mm_HandSolder" V 1280 1100 50  0001 C CNN
-F 3 "~" H 1350 1100 50  0001 C CNN
+F 0 "R1" V 1250 1100 50  0000 C CNN
+F 1 "1k" V 1350 1100 50  0000 C CNN
+F 2 "Resistor_SMD:R_0402_1005Metric_Pad0.72x0.64mm_HandSolder" V 1280 1100 50  0001 C CNN
+F 3 "https://www.te.com/commerce/DocumentDelivery/DDEController?Action=srchrtrv&DocNm=1773204-3&DocType=DS&DocLang=English" H 1350 1100 50  0001 C CNN
 F 4 "A130048TR-ND" H 1350 1100 50  0001 C CNN "Digi-Key_PN"
 F 5 "CRGCQ0402J1K0" H 1350 1100 50  0001 C CNN "MPN"
@@
 AR Path="/60306390/6030F0A9" Ref="R2"  Part="1"
 F 0 "R2" H 1620 946 50  0000 L CNN
-F 1 "501k" H 1620 855 50  0000 L CNN
+F 1 "505k" V 1550 800 50  0000 L CNN
 F 2 "Resistor_SMD:R_0805_2012Metric_Pad1.20x1.40mm_HandSolder" V 1480 900 50  0001 C CNN
-F 3 "~" H 1550 900 50  0001 C CNN
+F 3 "https://media.digikey.com/pdf/Data%20Sheets/KOA%20Speer/RN73R_Type_DS.pdf" H 1550 900 50  0001 C CNN
 F 4 "2019-RN73R2ATTD5053F100TR-ND" H 1550 900 50  0001 C CNN "Digi-Key_PN"
 F 5 "RN73R2ATTD5053F100" H 1550 900 50  0001 C CNN "MPN"
@@
 AR Path="/60306390/6030F0D1" Ref="R3"  Part="1"
 F 0 "R3" H 2020 1596 50  0000 L CNN
-F 1 "10k" H 2020 1505 50  0000 L CNN
+F 1 "10k" V 1950 1475 50  0000 L CNN
 F 2 "Resistor_SMD:R_0805_2012Metric_Pad1.20x1.40mm_HandSolder" V 1880 1550 50  0001 C CNN
-F 3 "~" H 1950 1550 50  0001 C CNN
+F 3 "https://www.susumu.co.jp/common/pdf/n_catalog_partition01_en.pdf" H 1950 1550 50  0001 C CNN
 F 4 "RG2012N-474-W-T1" H 1950 1550 50  0001 C CNN "Digi-Key_PN"
 F 5 "RG20N470KWTR-ND" H 1950 1550 50  0001 C CNN "MPN"

Commit message: Update ecad BOM
Change transistor to 2N4424
Parts:
- C1: footprint Capacitor_SMD:C_0402_1005Metric_Pad0.74x0.62mm_HandSolder -> Capacitor_SMD:C_0805_2012Metric_Pad1.18x1.45mm_HandSolder; MPN 399-C0402C224M8RACTUTR-ND -> GRM21B5C1H203JA01L
- Q1: value 2N4401BU -> 2N4424; MPN 2N4401-ND -> 2N4424; Spice_Lib_File ../lib/spice_models/2N4401.lib -> ../lib/spice_models/2N4424.lib; Spice_Model 2N4401 -> 2N4424
- R1: footprint Resistor_SMD:R_0402_1005Metric_Pad0.72x0.64mm_HandSolder -> Resistor_SMD:R_0805_2012Metric_Pad1.20x1.40mm_HandSolder; MPN CRGCQ0402J1K0 -> ERA6AEB102V
- R2: MPN RN73R2ATTD5053F100 -> ERJ-6ENF5103V
- R22: footprint Resistor_SMD:R_0402_1005Metric_Pad0.72x0.64mm_HandSolder -> Resistor_SMD:R_0805_2012Metric_Pad1.20x1.40mm_HandSolder; MPN ERJ-U02J155X -> ERJ-6ENF1004V
- R3: MPN RG20N470KWTR-ND -> ERJ-6GEYJ103V
Changed lines of the file:
@@
 F 0 "R22" H 820 1346 50  0000 L CNN
 F 1 "1M5" V 750 1225 50  0000 L CNN
-F 2 "Resistor_SMD:R_0402_1005Metric_Pad0.72x0.64mm_HandSolder" V 680 1300 50  0001 C CNN
-F 3 "https://industrial.panasonic.com/cdbs/www-data/pdf/RDP0000/AOA0000C334.pdf" H 750 1300 50  0001 C CNN
+F 2 "Resistor_SMD:R_0805_2012Metric_Pad1.20x1.40mm_HandSolder" V 680 1300 50  0001 C CNN
+F 3 "https://datasheet.octopart.com/ERJ-6ENF1004V-Panasonic-datasheet-5313456.pdf" H 750 1300 50  0001 C CNN
 F 4 "R" H 750 1300 50  0001 C CNN "Spice_Primitive"
 F 5 "1.5Meg" H 750 1300 50  0001 C CNN "Spice_Model"
 F 6 "Y" H 750 1300 50  0001 C CNN "Spice_Netlist_Enabled"
 F 7 "10-ERJ-U02J155XTR-ND" H 750 1300 50  0001 C CNN "Digi-Key_PN"
-F 8 "ERJ-U02J155X" H 750 1300 50  0001 C CNN "MPN"
+F 8 "ERJ-6ENF1004V" H 750 1300 50  0001 C CNN "MPN"
 	1    750  1300
 	1    0    0    -1
@@
 F 0 "C1" V 748 1100 50  0000 C CNN
 F 1 "20n" V 839 1100 50  0000 C CNN
-F 2 "Capacitor_SMD:C_0402_1005Metric_Pad0.74x0.62mm_HandSolder" H 1038 950 50  0001 C CNN
-F 3 "https://api.kemet.com/component-edge/download/datasheet/C0402C224M8RACTU.pdf" H 1000 1100 50  0001 C CNN
+F 2 "Capacitor_SMD:C_0805_2012Metric_Pad1.18x1.45mm_HandSolder" H 1038 950 50  0001 C CNN
+F 3 "https://datasheet.octopart.com/GRM21B5C1H203JA01L-Murata-datasheet-14402255.pdf" H 1000 1100 50  0001 C CNN
 F 4 "399-C0402C224M8RACTUTR-ND" H 1000 1100 50  0001 C CNN "Digi-Key_PN"
-F 5 "399-C0402C224M8RACTUTR-ND" H 1000 1100 50  0001 C CNN "MPN"
+F 5 "GRM21B5C1H203JA01L" H 1000 1100 50  0001 C CNN "MPN"
 	1    1000 1100
 	0    1    1    0
@@
 F 0 "R1" V 1250 1100 50  0000 C CNN
 F 1 "1k" V 1350 1100 50  0000 C CNN
-F 2 "Resistor_SMD:R_0402_1005Metric_Pad0.72x0.64mm_HandSolder" V 1280 1100 50  0001 C CNN
-F 3 "https://www.te.com/commerce/DocumentDelivery/DDEController?Action=srchrtrv&DocNm=1773204-3&DocType=DS&DocLang=English" H 1350 1100 50  0001 C CNN
+F 2 "Resistor_SMD:R_0805_2012Metric_Pad1.20x1.40mm_HandSolder" V 1280 1100 50  0001 C CNN
+F 3 "https://datasheet.octopart.com/ERA6AEB102V-Panasonic-datasheet-62287448.pdf" H 1350 1100 50  0001 C CNN
 F 4 "A130048TR-ND" H 1350 1100 50  0001 C CNN "Digi-Key_PN"
-F 5 "CRGCQ0402J1K0" H 1350 1100 50  0001 C CNN "MPN"
+F 5 "ERA6AEB102V" H 1350 1100 50  0001 C CNN "MPN"
 	1    1350 1100
 	0    1    1    0
@@
 F 1 "505k" V 1550 800 50  0000 L CNN
 F 2 "Resistor_SMD:R_0805_2012Metric_Pad1.20x1.40mm_HandSolder" V 1480 900 50  0001 C CNN
-F 3 "https://media.digikey.com/pdf/Data%20Sheets/KOA%20Speer/RN73R_Type_DS.pdf" H 1550 900 50  0001 C CNN
+F 3 "https://datasheet.octopart.com/ERJ-6ENF5103V-Panasonic-datasheet-13266541.pdf" H 1550 900 50  0001 C CNN
 F 4 "2019-RN73R2ATTD5053F100TR-ND" H 1550 900 50  0001 C CNN "Digi-Key_PN"
-F 5 "RN73R2ATTD5053F100" H 1550 900 50  0001 C CNN "MPN"
+F 5 "ERJ-6ENF5103V" H 1550 900 50  0001 C CNN "MPN"
 	1    1550 900
 	1    0    0    -1
@@
 AR Path="/60306390/6030F0C2" Ref="Q1"  Part="1"
 F 0 "Q1" H 1950 1450 60  0000 L CNN
-F 1 "2N4401BU" H 1950 1350 60  0000 L CNN
+F 1 "2N4424" H 1950 1350 60  0000 L CNN
 F 2 "digikey-footprints:TO-92-3" H 2050 1300 60  0001 L CNN
-F 3 "https://www.onsemi.com/pub/Collateral/MMBT4401-D.PDF" H 2050 1400 60  0001 L CNN
+F 3 "" H 2050 1400 60  0001 L CNN
 F 4 "2N4401-ND" H 2050 1500 60  0001 L CNN "Digi-Key_PN"
-F 5 "2N4401-ND" H 2050 1600 60  0001 L CNN "MPN"
+F 5 "2N4424" H 2050 1600 60  0001 L CNN "MPN"
 F 6 "Discrete Semiconductor Products" H 2050 1700 60  0001 L CNN "Category"
 F 7 "Transistors - Bipolar (BJT) - Single" H 2050 1800 60  0001 L CNN "Family"
@@
 F 12 "Active" H 2050 2300 60  0001 L CNN "Status"
 F 13 "Q" H 1850 1100 50  0001 C CNN "Spice_Primitive"
-F 14 "2N4401" H 1850 1100 50  0001 C CNN "Spice_Model"
+F 14 "2N4424" H 1850 1100 50  0001 C CNN "Spice_Model"
 F 15 "Y" H 1850 1100 50  0001 C CNN "Spice_Netlist_Enabled"
-F 16 "../lib/spice_models/2N4401.lib" H 1850 1100 50  0001 C CNN "Spice_Lib_File"
+F 16 "../lib/spice_models/2N4424.lib" H 1850 1100 50  0001 C CNN "Spice_Lib_File"
 F 17 "3 2 1" H 1850 1100 50  0001 C CNN "Spice_Node_Sequence"
 	1    1850 1100
@@
 F 1 "10k" V 1950 1475 50  0000 L CNN
 F 2 "Resistor_SMD:R_0805_2012Metric_Pad1.20x1.40mm_HandSolder" V 1880 1550 50  0001 C CNN
-F 3 "https://www.susumu.co.jp/common/pdf/n_catalog_partition01_en.pdf" H 1950 1550 50  0001 C CNN
+F 3 "https://datasheet.octopart.com/ERJ-6GEYJ103V-Panasonic-datasheet-13266872.pdf" H 1950 1550 50  0001 C CNN
 F 4 "RG2012N-474-W-T1" H 1950 1550 50  0001 C CNN "Digi-Key_PN"
-F 5 "RG20N470KWTR-ND" H 1950 1550 50  0001 C CNN "MPN"
+F 5 "ERJ-6GEYJ103V" H 1950 1550 50  0001 C CNN "MPN"
 	1    1950 1550
 	1    0    0    -1

Commit message: Library recovery
Parts:
- Q1: MPN 2N4424 -> 2N4401BU
Changed lines of the file:
@@
 F 1 "2N4424" H 1950 1350 60  0000 L CNN
 F 2 "digikey-footprints:TO-92-3" H 2050 1300 60  0001 L CNN
-F 3 "" H 2050 1400 60  0001 L CNN
+F 3 "https://www.onsemi.com/pub/Collateral/MMBT4401-D.PDF" H 2050 1400 60  0001 L CNN
 F 4 "2N4401-ND" H 2050 1500 60  0001 L CNN "Digi-Key_PN"
-F 5 "2N4424" H 2050 1600 60  0001 L CNN "MPN"
+F 5 "2N4401BU" H 2050 1600 60  0001 L CNN "MPN"
 F 6 "Discrete Semiconductor Products" H 2050 1700 60  0001 L CNN "Category"
 F 7 "Transistors - Bipolar (BJT) - Single" H 2050 1800 60  0001 L CNN "Family"

Commit message: Layout all components, first revision
Parts:
- Q1: footprint digikey-footprints:TO-92-3 -> digikey-footprints:TO-92-3_Formed_Leads
Changed lines of the file:
@@
 F 0 "Q1" H 1950 1450 60  0000 L CNN
 F 1 "2N4424" H 1950 1350 60  0000 L CNN
-F 2 "digikey-footprints:TO-92-3" H 2050 1300 60  0001 L CNN
+F 2 "digikey-footprints:TO-92-3_Formed_Leads" H 2050 1300 60  0001 L CNN
 F 3 "https://www.onsemi.com/pub/Collateral/MMBT4401-D.PDF" H 2050 1400 60  0001 L CNN
 F 4 "2N4401-ND" H 2050 1500 60  0001 L CNN "Digi-Key_PN"

Commit message: Change to using kicad-library submodule
Parts:
- Q1: Spice_Lib_File ../lib/spice_models/2N4424.lib -> ../lib/kicad-library/spice_models/2N4424.lib
Changed lines of the file:
@@
 F 14 "2N4424" H 1850 1100 50  0001 C CNN "Spice_Model"
 F 15 "Y" H 1850 1100 50  0001 C CNN "Spice_Netlist_Enabled"
-F 16 "../lib/spice_models/2N4424.lib" H 1850 1100 50  0001 C CNN "Spice_Lib_File"
+F 16 "../lib/kicad-library/spice_models/2N4424.lib" H 1850 1100 50  0001 C CNN "Spice_Lib_File"
 F 17 "3 2 1" H 1850 1100 50  0001 C CNN "Spice_Node_Sequence"
 	1    1850 1100
