File: ecad/MainBoard/volume.sch (KiCad schematic (older format))
At the start: 10 parts, among them Q2 2N4424

Commit message: PCB layout after data loss
Parts:
- Q2: footprint screaming-panda:TO-92-3_Formed_Leads -> digikey-footprints:TO-92-3
Changed lines of the file:
@@
 F 0 "Q2" H 2538 1453 60  0000 L CNN
 F 1 "2N4424" H 2538 1347 60  0000 L CNN
-F 2 "screaming-panda:TO-92-3_Formed_Leads" H 2550 1600 60  0001 L CNN
+F 2 "digikey-footprints:TO-92-3" H 2550 1600 60  0001 L CNN
 F 3 "https://my.centralsemi.com/datasheets/2N4424.PDF" H 2550 1700 60  0001 L CNN
 F 4 "2N4401-ND" H 2550 1800 60  0001 L CNN "Digi-Key_PN"

Commit message: Layout all components, first revision
Parts:
- Q2: footprint digikey-footprints:TO-92-3 -> digikey-footprints:TO-92-3_Formed_Leads
Changed lines of the file:
@@
 F 0 "Q2" H 2538 1453 60  0000 L CNN
 F 1 "2N4424" H 2538 1347 60  0000 L CNN
-F 2 "digikey-footprints:TO-92-3" H 2550 1600 60  0001 L CNN
+F 2 "digikey-footprints:TO-92-3_Formed_Leads" H 2550 1600 60  0001 L CNN
 F 3 "https://my.centralsemi.com/datasheets/2N4424.PDF" H 2550 1700 60  0001 L CNN
 F 4 "2N4401-ND" H 2550 1800 60  0001 L CNN "Digi-Key_PN"

Commit message: Change to using kicad-library submodule
Parts:
- Q2: Spice_Lib_File ../lib/spice_models/2N4424.lib -> ../lib/kicad-library/spice_models/2N4424.lib
- R21: Spice_Lib_File ../lib/spice_models/pots.lib -> ../lib/kicad-library/spice_models/pots.lib
Changed lines of the file:
@@
 F 11 "ON Semiconductor" H 2550 2500 60  0001 L CNN "Manufacturer"
 F 12 "Active" H 2550 2600 60  0001 L CNN "Status"
-F 13 "../lib/spice_models/2N4424.lib" H 2350 1400 50  0001 C CNN "Spice_Lib_File"
+F 13 "../lib/kicad-library/spice_models/2N4424.lib" H 2350 1400 50  0001 C CNN "Spice_Lib_File"
 F 14 "2N4424" H 2350 1400 50  0001 C CNN "Spice_Model"
 F 15 "Y" H 2350 1400 50  0001 C CNN "Spice_Netlist_Enabled"
@@
 F 5 "POTVolume" H 1550 1400 50  0001 C CNN "Spice_Model"
 F 6 "Y" H 1550 1400 50  0001 C CNN "Spice_Netlist_Enabled"
-F 7 "../lib/spice_models/pots.lib" H 1550 1400 50  0001 C CNN "Spice_Lib_File"
+F 7 "../lib/kicad-library/spice_models/pots.lib" H 1550 1400 50  0001 C CNN "Spice_Lib_File"
 F 8 "Volume Pot" H 1800 1650 50  0000 C CNN "Category"
 F 9 "75160-195-08LF" H 1550 1400 50  0001 C CNN "Digi-Key_PN"
